Commit message: 修复四轮驱动与Nav2导航，优化雷达避障并移除异常房门
- 修复 Gazebo 四轮差速驱动配置，使前后四轮共同驱动，解决机器人无法正常转向及里程计偏差问题。
- 调整机器人出生点至 (-1, 0)，同步 AMCL 初始定位，避免出生点靠近障碍物。
- 降低激光雷达高度，新增扫描自过滤功能，改善障碍物识别与导航代价地图。
- 完善 Nav2 导航参数、速度平滑与碰撞监测，验证全局路径规划及实际导航能够成功完成。
- 移除 101、102 房间异常门模型，修正对应静态地图，使房间入口保持常开。
- 清理门控制器启动逻辑，调整送药演示流程，更新相关测试及项目文档。

验证：四轮转向、TF定位及多次 Nav2 导航测试已通过；房门移除和地图调整已完成静态检查，待主机上重新构建并运行验收。

File: urdf/dual_arm_mobile_robot.urdf (robot description, URDF)
Before this commit: robot dual_arm_mobile_robot, 19 links, 18 joints
Links:
- added link camera_link, mass 0.15; collision box size=0.06 0.08 0.05; visual box size=0.06 0.08 0.05
- added link camera_optical_frame, mass 0.001; collision sphere radius=0.001; visual sphere radius=0.001
- added link laser_support, mass 0.1; collision cylinder length=0.03 radius=0.025; visual cylinder length=0.03 radius=0.025
- added link left_finger_left, mass 0.05; collision box size=0.025 0.01 0.08; visual box size=0.025 0.01 0.08
- added link left_finger_right, mass 0.05; collision box size=0.025 0.01 0.08; visual box size=0.025 0.01 0.08
- added link right_finger_left, mass 0.05; collision box size=0.025 0.01 0.08; visual box size=0.025 0.01 0.08
- added link right_finger_right, mass 0.05; collision box size=0.025 0.01 0.08; visual box size=0.025 0.01 0.08
- link left_forearm: mass 0.8 -> 0.5
- link left_gripper: mass 0.3 -> 0.2; geometry collision box size=0.06 0.06 0.04; visual box size=0.06 0.06 0.04
- link left_upper_arm: mass 1 -> 0.8
- link right_forearm: mass 0.8 -> 0.5
- link right_gripper: mass 0.3 -> 0.2; geometry collision box size=0.06 0.06 0.04; visual box size=0.06 0.06 0.04
- link right_upper_arm: mass 1 -> 0.8
- link torso: geometry collision box size=0.015 0.015 0.1; collision box size=0.015 0.015 0.1
Joints:
- added joint camera_link_joint: type fixed, parent torso, child camera_link, origin xyz=0.20 0 0.65 rpy=0 0 0
- added joint camera_optical_frame_joint: type fixed, parent camera_link, child camera_optical_frame, origin xyz=0 0 0 rpy=-1.57079632679 0 -1.57079632679
- added joint laser_support_joint: type fixed, parent base_link, child laser_support, origin xyz=0 0 0.235 rpy=0 0 0
- added joint left_finger_left_joint: type prismatic, parent left_gripper, child left_finger_left, origin xyz=0 0.008 -0.04 rpy=0 0 0, axis 0 1 0, limit lower=0 upper=0.025 effort=10 velocity=0.05
- added joint left_finger_right_joint: type prismatic, parent left_gripper, child left_finger_right, origin xyz=0 -0.008 -0.04 rpy=0 0 0, axis 0 -1 0, limit lower=0 upper=0.025 effort=10 velocity=0.05
- added joint right_finger_left_joint: type prismatic, parent right_gripper, child right_finger_left, origin xyz=0 0.008 -0.04 rpy=0 0 0, axis 0 1 0, limit lower=0 upper=0.025 effort=10 velocity=0.05
- added joint right_finger_right_joint: type prismatic, parent right_gripper, child right_finger_right, origin xyz=0 -0.008 -0.04 rpy=0 0 0, axis 0 -1 0, limit lower=0 upper=0.025 effort=10 velocity=0.05
- joint laser_joint: origin xyz=0.25 0 0.15 rpy=0 0 0 -> xyz=0 0 0.27 rpy=0 0 0
- joint left_elbow_joint: limit lower=0 upper=2.5 effort=30 velocity=1.0 -> lower=0 upper=2.5 effort=30 velocity=0.8
- joint left_forearm_joint: axis (none) -> 0 0 1; limit (none) -> lower=-3.14 upper=3.14 effort=20 velocity=0.8; type fixed -> revolute
- joint left_gripper_joint: axis (none) -> 0 0 1; limit (none) -> lower=-3.14 upper=3.14 effort=10 velocity=0.8; type fixed -> revolute
- joint left_shoulder_joint: limit lower=-1.57 upper=1.57 effort=50 velocity=1.0 -> lower=-1.57 upper=1.57 effort=50 velocity=0.8; origin xyz=0 0.2 0.5 rpy=0 0 0 -> xyz=0 0.32 0.5 rpy=0 0 0
- joint left_upper_arm_joint: limit lower=-3.14 upper=3.14 effort=50 velocity=1.0 -> lower=-1.57 upper=1.57 effort=50 velocity=0.8
- joint left_wrist_joint: axis 0 0 1 -> 0 1 0; limit lower=-1.57 upper=1.57 effort=20 velocity=1.0 -> lower=-1.57 upper=1.57 effort=20 velocity=0.8
- joint right_elbow_joint: limit lower=0 upper=2.5 effort=30 velocity=1.0 -> lower=0 upper=2.5 effort=30 velocity=0.8
- joint right_forearm_joint: axis (none) -> 0 0 1; limit (none) -> lower=-3.14 upper=3.14 effort=20 velocity=0.8; type fixed -> revolute
- joint right_gripper_joint: axis (none) -> 0 0 1; limit (none) -> lower=-3.14 upper=3.14 effort=10 velocity=0.8; type fixed -> revolute
- joint right_shoulder_joint: limit lower=-1.57 upper=1.57 effort=50 velocity=1.0 -> lower=-1.57 upper=1.57 effort=50 velocity=0.8; origin xyz=0 -0.2 0.5 rpy=0 0 0 -> xyz=0 -0.32 0.5 rpy=0 0 0
- joint right_upper_arm_joint: limit lower=-3.14 upper=3.14 effort=50 velocity=1.0 -> lower=-1.57 upper=1.57 effort=50 velocity=0.8
- joint right_wrist_joint: axis 0 0 1 -> 0 1 0; limit lower=-1.57 upper=1.57 effort=20 velocity=1.0 -> lower=-1.57 upper=1.57 effort=20 velocity=0.8
